File: PCB/motor-controller/motor-controller.kicad_pcb (KiCad board)
At the start: 2 copper layers, 100 x 100 mm, 70 parts, among them J1 POWER, J10 DIGITAL OUT3, J11 DIGITAL OUT4, J12 USB_B, J2 ANALOG OUT1, J3 ANALOG OUT2, J4 ANALOG INPUT, J5 ANALOG OUT3, J6 ANALOG OUT4, J7 DIGITAL INPUT, J8 DIGITAL OUT1, J9 DIGITAL OUT2, SW1 D1A, SW2 D1B, SW3 D2A, SW4 D2B, SW5 D3A, SW6 D3B, SW7 D4A, SW8 D4B, U1 74HC04, U10 74HC08, U11 74HC08, U12 74HC08, U2 74HC08, U3 74HC08, U4 74HC14, U5 74HC04, U6 74HC04, U7 74HC08, U8 74HC08, U9 74HC08

Commit message: 基板データ完成
git-svn-id: https://shiro-home.ddns.net/svn/project/motor-driver/trunk@6 73406841-da20-4056-b287-c5b29fcc9b8e
Parts:
- moved J7 1.27 mm to (103.8, 85.2)
- moved RN1 1.27 mm to (108.9, 82.7)
Connections:
- U8 pad 1: /DIN2A -> Net-(U5-Pad2)
- U8 pad 10: /OSC2 -> Net-(U8-Pad10)
- U8 pad 11: Net-(U8-Pad11) -> Net-(U8-Pad10)
- U8 pad 12: Net-(U5-Pad2) -> /DIN2A
- U8 pad 13: /DIN2B -> Net-(U5-Pad4)
- U8 pad 2: Net-(U5-Pad4) -> /DIN2B
- U8 pad 4: Net-(U8-Pad11) -> Net-(U5-Pad6)
- U8 pad 5: Net-(U8-Pad3) -> /OSC2
- U8 pad 6: Net-(U5-Pad5) -> Net-(U8-Pad6)
- U8 pad 8: Net-(U8-Pad8) -> Net-(U5-Pad5)
- U8 pad 9: Net-(U5-Pad6) -> Net-(U8-Pad3)
- U9 pad 10: Net-(U8-Pad3) -> Net-(U8-Pad10)
- U9 pad 12: Net-(U8-Pad11) -> Net-(U8-Pad3)
- U9 pad 13: Net-(U8-Pad8) -> Net-(U8-Pad6)
- U9 pad 9: Net-(U8-Pad8) -> Net-(U8-Pad6)
Routing:
- net Net-(U8-Pad6): track 0.00 -> 27.4 mm
- net Net-(U8-Pad11): track 26.0 -> 0.00 mm
- net Net-(U8-Pad8): track 19.6 -> 0.00 mm
- net Net-(U8-Pad10): track 0.00 -> 15.6 mm, vias 0 -> 1
- net Net-(U5-Pad5): track 34.6 -> 23.5 mm
- net Net-(U5-Pad4): track 21.9 -> 12.3 mm
- net Net-(U5-Pad2): track 25.0 -> 19.8 mm, vias 1 -> 0
- net /DIN4A: track 75.9 -> 81.0 mm
- net Net-(C5-Pad1): track 46.5 -> 43.4 mm, vias 1 -> 0
- net /OSC2: track 54.2 -> 51.1 mm
- net /PWM4IN: track 90.1 -> 87.3 mm
- net /DOUT1A: track 25.6 -> 28.3 mm
- net /DIN4B: track 86.5 -> 88.9 mm
- net /DIN2B: track 86.9 -> 89.1 mm, vias 2 -> 0
- net Net-(U7-Pad8): track 20.5 -> 22.5 mm
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Other:
- board text added: "5V"
- board text added: "@daisuke_ym 2020"
- board text added: "JLCJLCJLCJLC"
- board text added: "MOTOR CONTROLLER"
- board text added: "POWER"
- board text added: "SPEED"
