File: PCB/motor-controller/motor-controller.sch (KiCad schematic (older format))
At the start: 66 parts, among them J1 POWER, J10 DIGITAL OUT3, J11 DIGITAL OUT4, J12 USB_B, J2 ANALOG OUT1, J3 ANALOG OUT2, J4 ANALOG INPUT, J5 ANALOG OUT3, J6 ANALOG OUT4, J7 DIGITAL INPUT, J8 DIGITAL OUT1, J9 DIGITAL OUT2, SW1 D1A, SW2 D1B, SW3 D2A, SW4 D2B, SW5 D3A, SW6 D3B, SW7 D4A, SW8 D4B, U1 74HC04, U10 74HC08, U11 74HC08, U12 74HC08, U2 74HC08, U3 74HC08, U4 74HC14, U5 74HC04, U6 74HC04, U7 74HC08, U8 74HC08, U9 74HC08

Commit message: 基板データ完成
git-svn-id: https://shiro-home.ddns.net/svn/project/motor-driver/trunk@6 73406841-da20-4056-b287-c5b29fcc9b8e
Connections:
- net DIN2A: now also U8.12; no longer U8.1
- net DIN2B: now also U8.2; no longer U8.13
- net OSC2: now also U8.5; no longer U8.10
- net at U5.2: now also U8.1; no longer U8.12
- net at U5.4: now also U8.13; no longer U8.2
- net at U5.5: now also U8.8; no longer U8.6
- net at U9.13, U9.9: now also U8.6; no longer U8.8
- net at U5.6: now also U8.4; no longer U8.9
- new net: U8.3, U8.9, U9.12
- new net: U8.10, U8.11, U9.10
Changed lines of the file:
@@
 $Comp
 L 74xx:74LS08 U8
-U 4 1 5F7672E7
+U 1 1 5F7672E7
 P 9700 2800
 F 0 "U8" H 9700 3125 50  0000 C CNN
@@
 F 2 "Package_DIP:DIP-14_W7.62mm_Socket" H 9700 2800 50  0001 C CNN
 F 3 "https://assets.nexperia.com/documents/data-sheet/74HC_HCT04.pdf" H 9700 2800 50  0001 C CNN
-	4    9700 2800
+	1    9700 2800
 	1    0    0    -1
 $EndComp
@@
 $Comp
 L 74xx:74LS08 U8
-U 1 1 5F7672FB
+U 4 1 5F7672FB
 P 9700 3600
 F 0 "U8" H 9700 3925 50  0000 C CNN
@@
 F 2 "Package_DIP:DIP-14_W7.62mm_Socket" H 9700 3600 50  0001 C CNN
 F 3 "https://assets.nexperia.com/documents/data-sheet/74HC_HCT04.pdf" H 9700 3600 50  0001 C CNN
-	1    9700 3600
+	4    9700 3600
 	1    0    0    -1
 $EndComp
 $Comp
 L 74xx:74LS08 U8
-U 2 1 5F767305
+U 3 1 5F767305
 P 10300 3200
 F 0 "U8" H 10300 3525 50  0000 C CNN
@@
 F 2 "Package_DIP:DIP-14_W7.62mm_Socket" H 10300 3200 50  0001 C CNN
 F 3 "https://assets.nexperia.com/documents/data-sheet/74HC_HCT04.pdf" H 10300 3200 50  0001 C CNN
-	2    10300 3200
+	3    10300 3200
 	1    0    0    -1
 $EndComp
@@
 $Comp
 L 74xx:74LS08 U8
-U 3 1 5F767319
+U 2 1 5F767319
 P 11700 3300
 F 0 "U8" H 11700 3625 50  0000 C CNN
@@
 F 2 "Package_DIP:DIP-14_W7.62mm_Socket" H 11700 3300 50  0001 C CNN
 F 3 "https://assets.nexperia.com/documents/data-sheet/74HC_HCT04.pdf" H 11700 3300 50  0001 C CNN
-	3    11700 3300
+	2    11700 3300
 	1    0    0    -1
 $EndComp
