File: PCB/motor-driver5/motor-driver5.sch (KiCad schematic (older format))
At the start: 50 parts, among them J1 Motor Power, J2 Logic Power, J3 Input Ch1, J4 Input Ch2, M1 Motor_DC, M2 Motor_DC, Q1 Q_PMOS_GDS, Q2 Q_NMOS_GDS, Q3 Q_PMOS_GDS, Q4 Q_NMOS_GDS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

Commit message: 電源ラインが細かったので，基板サイズを大きくして太く修正した。
git-svn-id: https://shiro-home.ddns.net/svn/project/motor-driver/trunk@19 73406841-da20-4056-b287-c5b29fcc9b8e
Parts:
- C1, C2, C3, C4: footprint Capacitor_THT:CP_Radial_D5.0mm_P2.50mm -> Capacitor_THT:CP_Radial_D4.0mm_P1.50mm
Changed lines of the file:
@@
 F 0 "C1" H 1788 3696 50  0000 L CNN
 F 1 "10u" H 1788 3605 50  0000 L CNN
-F 2 "Capacitor_THT:CP_Radial_D5.0mm_P2.50mm" H 1700 3650 50  0001 C CNN
+F 2 "Capacitor_THT:CP_Radial_D4.0mm_P1.50mm" H 1700 3650 50  0001 C CNN
 F 3 "~" H 1700 3650 50  0001 C CNN
 	1    1700 3650
@@
 F 0 "C2" H 1788 4596 50  0000 L CNN
 F 1 "10u" H 1788 4505 50  0000 L CNN
-F 2 "Capacitor_THT:CP_Radial_D5.0mm_P2.50mm" H 1700 4550 50  0001 C CNN
+F 2 "Capacitor_THT:CP_Radial_D4.0mm_P1.50mm" H 1700 4550 50  0001 C CNN
 F 3 "~" H 1700 4550 50  0001 C CNN
 	1    1700 4550
@@
 F 0 "C3" H 1788 5696 50  0000 L CNN
 F 1 "10u" H 1788 5605 50  0000 L CNN
-F 2 "Capacitor_THT:CP_Radial_D5.0mm_P2.50mm" H 1700 5650 50  0001 C CNN
+F 2 "Capacitor_THT:CP_Radial_D4.0mm_P1.50mm" H 1700 5650 50  0001 C CNN
 F 3 "~" H 1700 5650 50  0001 C CNN
 	1    1700 5650
@@
 F 0 "C4" H 1788 6596 50  0000 L CNN
 F 1 "10u" H 1788 6505 50  0000 L CNN
-F 2 "Capacitor_THT:CP_Radial_D5.0mm_P2.50mm" H 1700 6550 50  0001 C CNN
+F 2 "Capacitor_THT:CP_Radial_D4.0mm_P1.50mm" H 1700 6550 50  0001 C CNN
 F 3 "~" H 1700 6550 50  0001 C CNN
 	1    1700 6550
