File: PCB/motor-driver4/motor-driver4.sch (KiCad schematic (older format))
At the start: 83 parts, among them J1 Motor Power, M1 Motor_DC, Q3 Q_NMOS_GDS

Commit message: ほぼ完成
git-svn-id: https://shiro-home.ddns.net/svn/project/motor-driver/trunk@12 73406841-da20-4056-b287-c5b29fcc9b8e
Parts:
- removed J?: Motor Power, Connector_JST:JST_VH_B2PS-VH_1x02_P3.96mm_Horizontal, symbol Connector_Generic:Conn_01x02
- removed J?: Logic Power, Connector_JST:JST_VH_B2PS-VH_1x02_P3.96mm_Horizontal, symbol Connector_Generic:Conn_01x02
- added C10, C11, C4, C5, C7, C8: 10u, Capacitor_THT:CP_Radial_D5.0mm_P2.50mm, symbol Device:CP_Small
- added C12, C3, C6, C9: 0.1u, Capacitor_THT:C_Disc_D3.4mm_W2.1mm_P2.50mm, symbol Device:C_Small
- added R11, R12, R21, R22, R31, R32: 4k7, Resistor_THT:R_Axial_DIN0207_L6.3mm_D2.5mm_P10.16mm_Horizontal, symbol Device:R
- added SW3, SW4, SW5, SW6, SW7, SW8: SW_Push, MyLib:TactSW_TVBP06_3.5x6.0-ThroughHole, symbol Switch:SW_Push
- added U2, U3, U4: ATtiny85-20PU, Package_DIP:DIP-8_W7.62mm, symbol MCU_Microchip_ATtiny:ATtiny85-20PU
- C1, C2: renamed from C?; footprint (none) -> Capacitor_THT:CP_Radial_D5.0mm_P2.50mm
- J2, J3, J4, J5, J6: renamed from J?; footprint Connector_JST:JST_VH_B2PS-VH_1x02_P3.96mm_Horizontal -> Connector_PinHeader_2.54mm:PinHeader_1x02_P2.54mm_Horizontal
- Q1, Q11, Q13, Q15, Q3, Q5, Q7, Q9: renamed from Q?; footprint (none) -> Package_TO_SOT_THT:TO-220-3_Horizontal_TabDown
- SW1, SW2: renamed from SW?; footprint (none) -> MyLib:TactSW_TVBP06_3.5x6.0-ThroughHole
- gave numbers to parts that had none: 59
- renumbered Q3 to Q2, R3 to R5, R7 to R6
Connections:
- net +5V: now also C12.1, C3.1, C6.1, C9.1, SW3.2, SW4.2, SW5.2, SW6.2, SW7.2, SW8.2, U2.8 (VCC), U3.8 (VCC), U4.8 (VCC)
- net GND: now also C10.2, C11.2, C12.2, C3.2, C4.2, C5.2, C6.2, C7.2, C8.2, C9.2, U2.4 (GND), U3.4 (GND), U4.4 (GND)
- net IN1A: now also J3.2 (Pin_2); no longer J3.1 (Pin_1)
- net IN1B: now also J3.1 (Pin_1); no longer J3.2 (Pin_2)
- net IN2A: now also J4.2 (Pin_2), R11.1, SW3.1; no longer J4.1 (Pin_1)
- net IN2B: now also J4.1 (Pin_1), R12.1, SW4.1; no longer J4.2 (Pin_2)
- net IN3A: now also J5.2 (Pin_2), R21.1, SW5.1; no longer J5.1 (Pin_1)
- net IN3B: now also J5.1 (Pin_1), R22.1, SW6.1; no longer J5.2 (Pin_2)
- net IN4A: now also J6.2 (Pin_2), R31.1, SW7.1; no longer J6.1 (Pin_1)
- net IN4B: now also J6.1 (Pin_1), R32.1, SW8.1; no longer J6.2 (Pin_2)
- net PC2A: now also R13.1, R18.1, U2.5 (AREF/PB0); no longer R23.1, R28.1
- net PC2B: now also R14.1, R17.1, U2.6 (PB1); no longer R24.1, R27.1
- net PC3A: now also R23.1, R28.1, U3.5 (AREF/PB0); no longer R13.1, R18.1
- net PC3B: now also R24.1, R27.1, U3.6 (PB1); no longer R14.1, R17.1
- net PC4A: now also U4.5 (AREF/PB0)
- net PC4B: now also U4.6 (PB1)
- new net IN2AA: C4.1, R11.2, U2.2 (XTAL1/PB3)
- new net IN2BA: C5.1, R12.2, U2.3 (XTAL2/PB4)
- new net IN3AA: C7.1, R21.2, U3.2 (XTAL1/PB3)
- new net IN3BA: C8.1, R22.2, U3.3 (XTAL2/PB4)
- new net IN4AA: C10.1, R31.2, U4.2 (XTAL1/PB3)
- new net IN4BA: C11.1, R32.2, U4.3 (XTAL2/PB4)
- no-connect marks 1 -> 8
Other:
- moved on the sheet: C1, C2, J1, J2, J3, J4, J5, J6, M1, M2, M3, M4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

Commit message: コンデンサのフットプリントを変更した
git-svn-id: https://shiro-home.ddns.net/svn/project/motor-driver/trunk@20 73406841-da20-4056-b287-c5b29fcc9b8e
Parts:
- C1, C10, C11, C2, C4, C5, C7, C8: footprint Capacitor_THT:CP_Radial_D5.0mm_P2.50mm -> Capacitor_THT:CP_Radial_D4.0mm_P1.50mm
Changed lines of the file:
@@
 F 0 "C1" H 3288 1496 50  0000 L CNN
 F 1 "10u" H 3288 1405 50  0000 L CNN
-F 2 "Capacitor_THT:CP_Radial_D5.0mm_P2.50mm" H 3200 1450 50  0001 C CNN
+F 2 "Capacitor_THT:CP_Radial_D4.0mm_P1.50mm" H 3200 1450 50  0001 C CNN
 F 3 "~" H 3200 1450 50  0001 C CNN
 	1    3200 1450
@@
 F 0 "C2" H 3288 2396 50  0000 L CNN
 F 1 "10u" H 3288 2305 50  0000 L CNN
-F 2 "Capacitor_THT:CP_Radial_D5.0mm_P2.50mm" H 3200 2350 50  0001 C CNN
+F 2 "Capacitor_THT:CP_Radial_D4.0mm_P1.50mm" H 3200 2350 50  0001 C CNN
 F 3 "~" H 3200 2350 50  0001 C CNN
 	1    3200 2350
@@
 F 0 "C4" H 6788 1496 50  0000 L CNN
 F 1 "10u" H 6788 1405 50  0000 L CNN
-F 2 "Capacitor_THT:CP_Radial_D5.0mm_P2.50mm" H 6700 1450 50  0001 C CNN
+F 2 "Capacitor_THT:CP_Radial_D4.0mm_P1.50mm" H 6700 1450 50  0001 C CNN
 F 3 "~" H 6700 1450 50  0001 C CNN
 	1    6700 1450
@@
 F 0 "C5" H 6788 2396 50  0000 L CNN
 F 1 "10u" H 6788 2305 50  0000 L CNN
-F 2 "Capacitor_THT:CP_Radial_D5.0mm_P2.50mm" H 6700 2350 50  0001 C CNN
+F 2 "Capacitor_THT:CP_Radial_D4.0mm_P1.50mm" H 6700 2350 50  0001 C CNN
 F 3 "~" H 6700 2350 50  0001 C CNN
 	1    6700 2350
@@
 F 0 "C7" H 10288 1496 50  0000 L CNN
 F 1 "10u" H 10288 1405 50  0000 L CNN
-F 2 "Capacitor_THT:CP_Radial_D5.0mm_P2.50mm" H 10200 1450 50  0001 C CNN
+F 2 "Capacitor_THT:CP_Radial_D4.0mm_P1.50mm" H 10200 1450 50  0001 C CNN
 F 3 "~" H 10200 1450 50  0001 C CNN
 	1    10200 1450
@@
 F 0 "C8" H 10288 2396 50  0000 L CNN
 F 1 "10u" H 10288 2305 50  0000 L CNN
-F 2 "Capacitor_THT:CP_Radial_D5.0mm_P2.50mm" H 10200 2350 50  0001 C CNN
+F 2 "Capacitor_THT:CP_Radial_D4.0mm_P1.50mm" H 10200 2350 50  0001 C CNN
 F 3 "~" H 10200 2350 50  0001 C CNN
 	1    10200 2350
@@
 F 0 "C10" H 13788 1496 50  0000 L CNN
 F 1 "10u" H 13788 1405 50  0000 L CNN
-F 2 "Capacitor_THT:CP_Radial_D5.0mm_P2.50mm" H 13700 1450 50  0001 C CNN
+F 2 "Capacitor_THT:CP_Radial_D4.0mm_P1.50mm" H 13700 1450 50  0001 C CNN
 F 3 "~" H 13700 1450 50  0001 C CNN
 	1    13700 1450
@@
 F 0 "C11" H 13788 2396 50  0000 L CNN
 F 1 "10u" H 13788 2305 50  0000 L CNN
-F 2 "Capacitor_THT:CP_Radial_D5.0mm_P2.50mm" H 13700 2350 50  0001 C CNN
+F 2 "Capacitor_THT:CP_Radial_D4.0mm_P1.50mm" H 13700 2350 50  0001 C CNN
 F 3 "~" H 13700 2350 50  0001 C CNN
 	1    13700 2350
