File: PCB/patch-board/patch-board.sch (KiCad schematic (older format))
At the start: 96 parts, among them J1 USB_B, J11 ANALOG OUT1, J12 ANALOG OUT2, J13 ANALOG OUT3, J14 ANALOG OUT4, J15 ANALOG OUT1, J16 ANALOG OUT2, J17 ANALOG OUT3, J18 ANALOG OUT4, J2 POWER, J21 DIGITAL OUT1, J22 DIGITAL OUT2, J23 DIGITAL OUT3, J24 DIGITAL OUT4, J3 MEGA_13-8, J31 S01, J32 S02, J33 S03, J34 S04, J35 S05, J36 S06, J37 S07, J38 S08, J39 S09, J4 MEGA_7-0, J40 S10, J41 SV, J42 SV, J43 SV, J44 SV, J45 SV, J46 SV, J5 MEGA_14-21, J6 MEGA_A8-A15, J7 MEGA_22-53, J8 Conn_01x02, SW1 D1A, SW11 SW_DPST, SW12 SW_DPST, SW2 D1B, SW3 D2A, SW4 D2B, SW5 D3A, SW6 D3B, SW7 D4A, SW8 D4B, U1 74HC00, U10 74HC08, U11 74HC00, U12 74HC08, U13 74HC08, U2 74HC08, U3 74HC08, U4 74HC00, U5 74HC08, U6 74HC08, U7 74HC14, U8 74HC00, U9 74HC08

Commit message: まだ途中
git-svn-id: https://shiro-home.ddns.net/svn/project/motor-driver/trunk@22 73406841-da20-4056-b287-c5b29fcc9b8e
Parts:
- removed J2: POWER, Connector_PinHeader_2.54mm:PinHeader_1x02_P2.54mm_Vertical, symbol Connector_Generic:Conn_01x02
- added J2: LOGIC POWER SUPPLY, Connector_PinHeader_2.54mm:PinHeader_2x05_P2.54mm_Vertical, symbol Connector_Generic:Conn_02x05_Odd_Even
- added J7: MEGA_A0-A7, Connector_PinHeader_2.54mm:PinHeader_1x08_P2.54mm_Vertical, symbol Connector_Generic:Conn_01x08
- added J8: MEGA_POWER, Connector_PinHeader_2.54mm:PinHeader_1x06_P2.54mm_Vertical, symbol Connector_Generic:Conn_01x06
- added R10, R5, R6, R7, R8, R9: 1k, Resistor_THT:R_Axial_DIN0207_L6.3mm_D2.5mm_P10.16mm_Horizontal, symbol Device:R
- C1, C10, C11, C12, C13, C2, C20, C21, C22, C23, C24, C3, C4, C5, C6, C7, C8, C9: footprint (none) -> Capacitor_THT:C_Disc_D3.4mm_W2.1mm_P2.50mm
- D11, D12: footprint (none) -> LED_THT:LED_D5.0mm-4_RGB
- J11: value ANALOG OUT1 -> AOUT1; footprint Connector_PinHeader_2.54mm:PinHeader_1x04_P2.54mm_Vertical -> Connector_PinHeader_2.54mm:PinHeader_1x02_P2.54mm_Vertical; symbol Connector_Generic:Conn_01x04 -> Connector_Generic:Conn_01x02
- J12: value ANALOG OUT2 -> AOUT2; footprint Connector_PinHeader_2.54mm:PinHeader_1x04_P2.54mm_Vertical -> Connector_PinHeader_2.54mm:PinHeader_1x02_P2.54mm_Vertical; symbol Connector_Generic:Conn_01x04 -> Connector_Generic:Conn_01x02
- J13: value ANALOG OUT3 -> AOUT3; footprint Connector_PinHeader_2.54mm:PinHeader_1x04_P2.54mm_Vertical -> Connector_PinHeader_2.54mm:PinHeader_1x02_P2.54mm_Vertical; symbol Connector_Generic:Conn_01x04 -> Connector_Generic:Conn_01x02
- J14: value ANALOG OUT4 -> AOUT4; footprint Connector_PinHeader_2.54mm:PinHeader_1x04_P2.54mm_Vertical -> Connector_PinHeader_2.54mm:PinHeader_1x02_P2.54mm_Vertical; symbol Connector_Generic:Conn_01x04 -> Connector_Generic:Conn_01x02
- J15: value ANALOG OUT1 -> AOUT5; footprint Connector_PinHeader_2.54mm:PinHeader_1x04_P2.54mm_Vertical -> Connector_PinHeader_2.54mm:PinHeader_1x02_P2.54mm_Vertical; symbol Connector_Generic:Conn_01x04 -> Connector_Generic:Conn_01x02
- J16: value ANALOG OUT2 -> AOUT6; footprint Connector_PinHeader_2.54mm:PinHeader_1x04_P2.54mm_Vertical -> Connector_PinHeader_2.54mm:PinHeader_1x02_P2.54mm_Vertical; symbol Connector_Generic:Conn_01x04 -> Connector_Generic:Conn_01x02
- J17: value ANALOG OUT3 -> AOUT7; footprint Connector_PinHeader_2.54mm:PinHeader_1x04_P2.54mm_Vertical -> Connector_PinHeader_2.54mm:PinHeader_1x02_P2.54mm_Vertical; symbol Connector_Generic:Conn_01x04 -> Connector_Generic:Conn_01x02
- J18: value ANALOG OUT4 -> AOUT8; footprint Connector_PinHeader_2.54mm:PinHeader_1x04_P2.54mm_Vertical -> Connector_PinHeader_2.54mm:PinHeader_1x02_P2.54mm_Vertical; symbol Connector_Generic:Conn_01x04 -> Connector_Generic:Conn_01x02
- J21, J22, J23, J24: footprint Connector_PinHeader_2.54mm:PinHeader_1x04_P2.54mm_Vertical -> Connector_PinHeader_2.54mm:PinHeader_1x02_P2.54mm_Vertical; symbol Connector_Generic:Conn_01x04 -> Connector_Generic:Conn_01x02
- J31, J32, J33, J34, J35, J36, J37, J38, J39, J41, J42, J43, J44, J45, J46: footprint (none) -> Connector_PinHeader_2.54mm:PinHeader_1x03_P2.54mm_Vertical
- J40: footprint (none) -> Connector_PinHeader_2.54mm:PinHeader_1x06_P2.54mm_Vertical
- J9: renamed from J7; footprint (none) -> Connector_PinHeader_2.54mm:PinHeader_2x18_P2.54mm_Vertical
- RV1, RV2, RV3, RV4: footprint MyLib:TSR-065 -> MyLib:GF063P1
- SW11, SW12: footprint (none) -> MyLib:DTS-6-V-2
- SW13: renamed from J8; footprint (none) -> Connector_PinHeader_2.54mm:PinHeader_1x02_P2.54mm_Vertical
- U1, U11, U4, U8: footprint (none) -> Package_SO:SO-14_5.3x10.2mm_P1.27mm
- U10, U12, U13, U2, U3, U5, U6, U7, U9: footprint Package_DIP:DIP-14_W7.62mm_Socket -> Package_SO:SO-14_5.3x10.2mm_P1.27mm
Connections:
- net +5V: now also J2.1 (Pin_1), J2.3 (Pin_3), J2.5 (Pin_5), J2.7 (Pin_7), J2.9 (Pin_9)
- net AOUT1A: now also U5.8; no longer U2.11
- net AOUT1B: now also J11.1 (Pin_1), U5.6; no longer J11.3 (Pin_3), U2.3
- net AOUT2A: now also U5.11; no longer U2.8
- net AOUT2B: now also J12.1 (Pin_1), U5.3; no longer J12.3 (Pin_3), U2.6
- net AOUT3A: now also U2.8; no longer U3.11
- net AOUT3B: now also J13.1 (Pin_1), U2.6; no longer J13.3 (Pin_3), U3.3
- net AOUT4A: now also U2.11; no longer U3.8
- net AOUT4B: now also J14.1 (Pin_1), U2.3; no longer J14.3 (Pin_3), U3.6
- net AOUT5A: now also U3.11; no longer U5.11
- net AOUT5B: now also J15.1 (Pin_1), U3.3; no longer J15.3 (Pin_3), U5.3
- net AOUT6A: now also U3.8; no longer U5.8
- net AOUT6B: now also J16.1 (Pin_1), U3.6; no longer J16.3 (Pin_3), U5.6
- net AOUT7B: now also J17.1 (Pin_1); no longer J17.3 (Pin_3)
- net AOUT8B: now also J18.1 (Pin_1); no longer J18.3 (Pin_3)
- net CSENSOR: now also J9.15 (Pin_15); no longer J9.23 (Pin_23)
- net DIN1A: now also J9.14 (Pin_14), U8.12, U8.13, U9.13; no longer J6.1 (Pin_1), U8.1, U8.2, U9.12
- net DIN1B: now also J9.16 (Pin_16), U8.10, U8.9; no longer J6.2 (Pin_2), U8.4, U8.5
- net DIN2A: now also J9.18 (Pin_18), U10.13, U8.4, U8.5; no longer J6.3 (Pin_3), U10.12, U8.10, U8.9
- net DIN2B: now also J9.20 (Pin_20), U10.1, U8.1, U8.2; no longer J6.4 (Pin_4), U10.2, U8.12, U8.13
- net DIN3A: now also J9.22 (Pin_22); no longer J6.5 (Pin_5)
- net DIN3B: now also J9.24 (Pin_24); no longer J6.6 (Pin_6)
- net DIN4A: now also J9.26 (Pin_26); no longer J6.7 (Pin_7)
- net DIN4B: now also J9.28 (Pin_28); no longer J6.8 (Pin_8)
- net DOUT1A: now also J21.1 (Pin_1); no longer J21.2 (Pin_2)
- net DOUT1B: now also J21.2 (Pin_2); no longer J21.3 (Pin_3)
- net DOUT2A: now also J22.1 (Pin_1); no longer J22.2 (Pin_2)
- net DOUT2B: now also J22.2 (Pin_2); no longer J22.3 (Pin_3)
- net DOUT3A: now also J23.1 (Pin_1); no longer J23.2 (Pin_2)
- net DOUT3B: now also J23.2 (Pin_2); no longer J23.3 (Pin_3)
- net DOUT4A: now also J24.1 (Pin_1); no longer J24.2 (Pin_2)
- net DOUT4B: now also J24.2 (Pin_2); no longer J24.3 (Pin_3)
- net GND: now also J2.10 (Pin_10), J2.2 (Pin_2), J2.4 (Pin_4), J2.6 (Pin_6), J2.8 (Pin_8), J8.4 (Pin_4), J8.5 (Pin_5); no longer J11.1 (Pin_1), J11.4 (Pin_4), J12.1 (Pin_1), J12.4 (Pin_4), J13.1 (Pin_1), J13.4 (Pin_4), J14.1 (Pin_1), J14.4 (Pin_4), J15.1 (Pin_1), J15.4 (Pin_4), J16.1 (Pin_1), J16.4 (Pin_4), J17.1 (Pin_1), J17.4 (Pin_4), J18.1 (Pin_1), J18.4 (Pin_4), J21.1 (Pin_1), J21.4 (Pin_4), J22.1 (Pin_1), J22.4 (Pin_4), J23.1 (Pin_1), J23.4 (Pin_4), J24.1 (Pin_1), J24.4 (Pin_4)
- net LED1B: now also J9.9 (Pin_9), R7.2; no longer D11.3 (BA), J9.7 (Pin_7)
- net LED1G: now also J9.7 (Pin_7), R6.2; no longer D11.4 (GA), J9.5 (Pin_5)
- net LED1R: now also J9.5 (Pin_5), R5.2; no longer D11.1 (RA), J9.3 (Pin_3)
- net LED2B: now also J9.12 (Pin_12), R10.2; no longer D12.3 (BA), J9.8 (Pin_8)
- net LED2G: now also J9.10 (Pin_10), R9.2; no longer D12.4 (GA), J9.6 (Pin_6)
- net LED2R: now also J9.8 (Pin_8), R8.2; no longer D12.1 (RA), J9.4 (Pin_4)
- net LSENSOR: now also J9.17 (Pin_17); no longer J9.24 (Pin_24)
- net OSC1: now also U7.12; no longer U7.2
- net OSC2: now also U7.10; no longer U7.4
- net OSC3: now also U7.4; no longer U7.12
- net OSC4: now also U7.2; no longer U7.10
- net PWM1IN: now also U5.10, U5.4; no longer U2.13, U2.2
- net PWM2IN: now also U5.1, U5.13; no longer U2.10, U2.5
- net PWM3IN: now also U2.10, U2.4; no longer U3.13, U3.2
- net PWM4IN: now also U2.1, U2.13; no longer U3.10, U3.5
- net PWM5IN: now also U3.1, U3.13; no longer U5.13, U5.2
- net PWM6IN: now also U3.10, U3.4; no longer U5.10, U5.5
- net PWM7IN: now also U6.1; no longer U6.2
- net PWM8IN: now also U6.4; no longer U6.5
- net RSENSOR: now also J9.13 (Pin_13); no longer J9.22 (Pin_22)
- net SEL1: now also U4.10, U4.9, U5.9; no longer U1.1, U1.2, U2.12
- net SEL2: now also U4.12, U4.13, U5.12; no longer U1.4, U1.5, U2.9
- net SEL3: now also U2.9; no longer U3.12
- net SEL4: now also U2.12; no longer U3.9
- net SEL5: now also U1.1, U1.2, U3.12; no longer U4.1, U4.2, U5.12
- net SEL6: now also U1.4, U1.5, U3.9; no longer U4.4, U4.5, U5.9
- net SEL7: now also U4.1, U4.2; no longer U4.10, U4.9
- net SEL8: now also U4.4, U4.5; no longer U4.12, U4.13
- net SENSOR01: now also J6.1 (Pin_1); no longer J9.11 (Pin_11)
- net SENSOR02: now also J6.2 (Pin_2); no longer J9.12 (Pin_12)
- net SENSOR03: now also J6.3 (Pin_3); no longer J9.13 (Pin_13)
- net SENSOR04: now also J6.4 (Pin_4); no longer J9.14 (Pin_14)
- net SENSOR05: now also J6.5 (Pin_5); no longer J9.15 (Pin_15)
- net SENSOR06: now also J6.6 (Pin_6); no longer J9.16 (Pin_16)
- net SENSOR07: now also J6.7 (Pin_7); no longer J9.17 (Pin_17)
- net SENSOR08: now also J6.8 (Pin_8); no longer J9.18 (Pin_18)
- net SENSOR09: now also J9.30 (Pin_30); no longer J9.19 (Pin_19)
- net SV1: now also J9.19 (Pin_19); no longer J9.25 (Pin_25)
- net SV2: now also J9.21 (Pin_21); no longer J9.26 (Pin_26)
- net SV3: now also J9.23 (Pin_23); no longer J9.27 (Pin_27)
- net SV4: now also J9.25 (Pin_25); no longer J9.28 (Pin_28)
- net SV5: now also J9.27 (Pin_27); no longer J9.29 (Pin_29)
- net SV6: now also J9.29 (Pin_29); no longer J9.30 (Pin_30)
- net SW11: now also J9.3 (Pin_3); no longer J9.9 (Pin_9)
- net SW12: now also J9.6 (Pin_6); no longer J9.10 (Pin_10)
- net WSENSOR: now also J9.11 (Pin_11); no longer J9.21 (Pin_21)
- net at U1.3: now also U3.2; no longer U2.1
- net at U1.6: now also U3.5; no longer U2.4
- net at U1.8: now also U2.5; no longer U3.1
- net at U1.11: now also U2.2; no longer U3.4
- net at C21.1, R1.2: now also U7.13; no longer U7.1
- net at U9.1: now also U8.11; no longer U8.3
- net at U8.6: now also U10.2; no longer U9.13
- net at C22.1, R2.2: now also U7.11; no longer U7.3
- net at U8.8: now also U9.12; no longer U10.1
- net at C23.1, R3.2: now also U7.3; no longer U7.13
- net at C24.1, R4.2: now also U7.1; no longer U7.11
- net at U4.3: now also U6.2; no longer U5.1
- net at U4.6: now also U6.5; no longer U5.4
- net at U4.8: now also U5.5; no longer U6.1
- net at U4.11: now also U5.2; no longer U6.4
- net GPIN renamed SW13
- net SW13: now also J9.4 (Pin_4); no longer J9.20 (Pin_20)
- new net: U10.12, U8.3
- new net: D11.1 (RA), R5.1
- new net: D11.4 (GA), R6.1
- new net: D11.3 (BA), R7.1
- new net: D12.1 (RA), R8.1
- new net: D12.4 (GA), R9.1
- new net: D12.3 (BA), R10.1
- no-connect marks 17 -> 29
Other:
- moved on the sheet: C20, D11, D12, J6, RN1, SW13, U1A, U1B, U1C, U1D, U2A, U2B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
