File: PCB/patch-board/patch-board.kicad_pcb (KiCad board)
At the start: 2 copper layers, 230 x 63 mm, 108 parts, among them J1 USB_B, J11 AOUT1, J12 AOUT2, J13 AOUT3, J14 AOUT4, J15 AOUT5, J16 AOUT6, J17 AOUT7, J18 AOUT8, J2 LOGIC POWER SUPPLY, J21 DIGITAL OUT1, J22 DIGITAL OUT2, J23 DIGITAL OUT3, J24 DIGITAL OUT4, J3 MEGA_13-8, J31 S01, J32 S02, J33 S03, J34 S04, J35 S05, J36 S06, J37 S07, J38 S08, J39 S09, J4 MEGA_7-0, J40 S10, J41 SV, J42 SV, J43 SV, J44 SV, J45 SV, J46 SV, J5 MEGA_14-21, J6 MEGA_A8-A15, J7 MEGA_A0-A7, J8 MEGA_POWER, J9 MEGA_22-53, SW1 D1A, SW11 SW_DPST, SW12 SW_DPST, SW13 Conn_01x02, SW2 D1B, SW3 D2A, SW4 D2B, SW5 D3A, SW6 D3B, SW7 D4A, SW8 D4B, U1 74HC00, U10 74HC08, U11 74HC00, U12 74HC08, U13 74HC08, U2 74HC08, U3 74HC08, U4 74HC00, U5 74HC08, U6 74HC08, U7 74HC14, U8 74HC00, U9 74HC08

Commit message: D13 ピンの配線ミスを修正 AOUT5-8 のシルクミスを修正 U13 のユニット割り当てミスを修正
git-svn-id: https://shiro-home.ddns.net/svn/project/motor-driver/trunk@32 73406841-da20-4056-b287-c5b29fcc9b8e
Parts:
- C21, C22, C23, C24: value 0.1u -> 1u
- R1, R2, R3, R4: value R -> 330
- RV1, RV2, RV3, RV4: value R_POT -> 5k
Connections:
- J3 pad 1: /PWM1IN -> Net-(J3-Pad1)
- J3 pad 3: Net-(J3-Pad3) -> /PWM1IN
Routing:
- net /PWM1IN: track 24.4 -> 29.5 mm
Other:
- board text added: "Rev.2"
