File: PCB/patch-board2022a/patch-board2022a.sch (KiCad schematic (older format))
At the start: 116 parts, among them J1 USB_B, J10 SERVO POWER SUPPLY, J11 AOUT1, J12 AOUT2, J13 AOUT3, J14 AOUT4, J15 AOUT5, J16 AOUT6, J17 AOUT7, J18 AOUT8, J2 LOGIC POWER SUPPLY, J21 DIGITAL OUT1, J22 DIGITAL OUT2, J23 DIGITAL OUT3, J24 DIGITAL OUT4, J3 MEGA_13-8, J31 S01, J32 S02, J33 S03, J34 S04, J35 S05, J36 S06, J37 S07, J38 S08, J39 S09, J4 MEGA_7-0, J41 SV, J42 SV, J43 SV, J44 SV, J45 SV, J46 SV, J5 MEGA_14-21, J6 MEGA_A8-A15, J7 MEGA_A0-A7, J8 MEGA_POWER, J9 MEGA_22-53, SW1 D1A, SW11 SW_DPST, SW12 SW_DPST, SW13 Conn_01x02, SW2 D1B, SW3 D2A, SW4 D2B, SW5 D3A, SW6 D3B, SW7 D4A, SW8 D4B, U1 74HC00, U10 74HC08, U11 74HC00, U12 74HC08, U13 74HC08, U14 TLP785, U15 TLP785, U16 TLP785, U17 TLP785, U18 TLP785, U19 TLP785, U2 74HC08, U3 74HC08, U4 74HC00, U5 74HC08, U6 74HC08, U7 74HC14, U8 74HC00, U9 74HC08

Commit message: 一応完成
git-svn-id: https://shiro-home.ddns.net/svn/project/motor-driver/trunk@40 73406841-da20-4056-b287-c5b29fcc9b8e
Parts:
- removed J11: AOUT1, Connector_PinHeader_2.54mm:PinHeader_1x02_P2.54mm_Vertical, symbol Connector_Generic:Conn_01x02
- removed J12: AOUT2, Connector_PinHeader_2.54mm:PinHeader_1x02_P2.54mm_Vertical, symbol Connector_Generic:Conn_01x02
- removed J13: AOUT3, Connector_PinHeader_2.54mm:PinHeader_1x02_P2.54mm_Vertical, symbol Connector_Generic:Conn_01x02
- removed J14: AOUT4, Connector_PinHeader_2.54mm:PinHeader_1x02_P2.54mm_Vertical, symbol Connector_Generic:Conn_01x02
- removed J15: AOUT5, Connector_PinHeader_2.54mm:PinHeader_1x02_P2.54mm_Vertical, symbol Connector_Generic:Conn_01x02
- removed J16: AOUT6, Connector_PinHeader_2.54mm:PinHeader_1x02_P2.54mm_Vertical, symbol Connector_Generic:Conn_01x02
- removed J17: AOUT7, Connector_PinHeader_2.54mm:PinHeader_1x02_P2.54mm_Vertical, symbol Connector_Generic:Conn_01x02
- removed J18: AOUT8, Connector_PinHeader_2.54mm:PinHeader_1x02_P2.54mm_Vertical, symbol Connector_Generic:Conn_01x02
- removed J21: DIGITAL OUT1, Connector_PinHeader_2.54mm:PinHeader_1x02_P2.54mm_Vertical, symbol Connector_Generic:Conn_01x02
- removed J22: DIGITAL OUT2, Connector_PinHeader_2.54mm:PinHeader_1x02_P2.54mm_Vertical, symbol Connector_Generic:Conn_01x02
- removed J23: DIGITAL OUT3, Connector_PinHeader_2.54mm:PinHeader_1x02_P2.54mm_Vertical, symbol Connector_Generic:Conn_01x02
- removed J24: DIGITAL OUT4, Connector_PinHeader_2.54mm:PinHeader_1x02_P2.54mm_Vertical, symbol Connector_Generic:Conn_01x02
- removed J39: S09, Connector_PinHeader_2.54mm:PinHeader_1x03_P2.54mm_Vertical, symbol Connector_Generic:Conn_01x03
- added J11: AOUT1, Connector_PinHeader_2.54mm:PinHeader_1x03_P2.54mm_Vertical, symbol Connector_Generic:Conn_01x03
- added J12: AOUT2, Connector_PinHeader_2.54mm:PinHeader_1x03_P2.54mm_Vertical, symbol Connector_Generic:Conn_01x03
- added J13: AOUT3, Connector_PinHeader_2.54mm:PinHeader_1x03_P2.54mm_Vertical, symbol Connector_Generic:Conn_01x03
- added J14: AOUT4, Connector_PinHeader_2.54mm:PinHeader_1x03_P2.54mm_Vertical, symbol Connector_Generic:Conn_01x03
- added J15: AOUT5, Connector_PinHeader_2.54mm:PinHeader_1x03_P2.54mm_Vertical, symbol Connector_Generic:Conn_01x03
- added J16: AOUT6, Connector_PinHeader_2.54mm:PinHeader_1x03_P2.54mm_Vertical, symbol Connector_Generic:Conn_01x03
- added J17: AOUT7, Connector_PinHeader_2.54mm:PinHeader_1x03_P2.54mm_Vertical, symbol Connector_Generic:Conn_01x03
- added J18: AOUT8, Connector_PinHeader_2.54mm:PinHeader_1x03_P2.54mm_Vertical, symbol Connector_Generic:Conn_01x03
- added J21: DOUT1, Connector_PinHeader_2.54mm:PinHeader_1x03_P2.54mm_Vertical, symbol Connector_Generic:Conn_01x03
- added J22: DOUT2, Connector_PinHeader_2.54mm:PinHeader_1x03_P2.54mm_Vertical, symbol Connector_Generic:Conn_01x03
- added J23: DOUT3, Connector_PinHeader_2.54mm:PinHeader_1x03_P2.54mm_Vertical, symbol Connector_Generic:Conn_01x03
- added J24: DOUT4, Connector_PinHeader_2.54mm:PinHeader_1x03_P2.54mm_Vertical, symbol Connector_Generic:Conn_01x03
Connections:
- net SENSOR9 is gone; now on net DIN1A: J9.12 (Pin_12)
- net AOUT1A: now also J11.3 (Pin_3)
- net AOUT1B: now also J11.1 (Pin_1)
- net AOUT2A: now also J12.3 (Pin_3)
- net AOUT2B: now also J12.1 (Pin_1)
- net AOUT3A: now also J13.3 (Pin_3)
- net AOUT3B: now also J13.1 (Pin_1)
- net AOUT4A: now also J14.3 (Pin_3)
- net AOUT4B: now also J14.1 (Pin_1)
- net AOUT5A: now also J15.3 (Pin_3)
- net AOUT5B: now also J15.1 (Pin_1)
- net AOUT6A: now also J16.3 (Pin_3)
- net AOUT6B: now also J16.1 (Pin_1)
- net AOUT7A: now also J17.3 (Pin_3)
- net AOUT7B: now also J17.1 (Pin_1)
- net AOUT8A: now also J18.3 (Pin_3)
- net AOUT8B: now also J18.1 (Pin_1)
- net DIN1A: no longer J9.14 (Pin_14)
- net DIN1B: now also J9.14 (Pin_14); no longer J9.16 (Pin_16)
- net DIN2A: now also J9.16 (Pin_16); no longer J9.18 (Pin_18)
- net DIN2B: now also J9.18 (Pin_18); no longer J9.20 (Pin_20)
- net DIN3A: now also J9.20 (Pin_20); no longer J9.22 (Pin_22)
- net DIN3B: now also J9.22 (Pin_22); no longer J9.24 (Pin_24)
- net DIN4A: now also J9.24 (Pin_24); no longer J9.26 (Pin_26)
- net DIN4B: now also J9.26 (Pin_26); no longer J9.28 (Pin_28)
- net DOUT1A: now also J21.3 (Pin_3)
- net DOUT1B: now also J21.1 (Pin_1)
- net DOUT2A: now also J22.3 (Pin_3)
- net DOUT2B: now also J22.1 (Pin_1)
- net DOUT3A: now also J23.3 (Pin_3)
- net DOUT3B: now also J23.1 (Pin_1)
- net DOUT4A: now also J24.3 (Pin_3)
- net DOUT4B: now also J24.1 (Pin_1)
- net LED1: now also J9.10 (Pin_10); no longer J9.5 (Pin_5)
- net SENSOR1: now also J6.1 (Pin_1); no longer J9.7 (Pin_7)
- net SENSOR2: now also J6.2 (Pin_2); no longer J9.9 (Pin_9)
- net SENSOR3: now also J6.3 (Pin_3); no longer J9.11 (Pin_11)
- net SENSOR4: now also J6.4 (Pin_4); no longer J9.13 (Pin_13)
- net SENSOR5: now also J6.5 (Pin_5); no longer J9.15 (Pin_15)
- net SENSOR6: now also J6.6 (Pin_6); no longer J9.17 (Pin_17)
- net SENSOR7: now also J6.7 (Pin_7); no longer J9.8 (Pin_8)
- net SENSOR8: now also J6.8 (Pin_8); no longer J9.10 (Pin_10)
- net SV1IN: now also J9.7 (Pin_7); no longer J9.19 (Pin_19)
- net SV2IN: now also J9.9 (Pin_9); no longer J9.21 (Pin_21)
- net SV3IN: now also J9.11 (Pin_11); no longer J9.23 (Pin_23)
- net SV4IN: now also J9.13 (Pin_13); no longer J9.25 (Pin_25)
- net SV5IN: now also J9.15 (Pin_15); no longer J9.27 (Pin_27)
- net SV6IN: now also J9.17 (Pin_17); no longer J9.29 (Pin_29)
- net SW12: now also J9.5 (Pin_5); no longer J9.6 (Pin_6)
- net DOUT4M: now reaches J9.30 (Pin_30)
- net DOUT4M: now also J24.2 (Pin_2)
- net AOUT8M: now reaches J7.1 (Pin_1)
- net AOUT8M: now also J18.2 (Pin_2)
- net AOUT7M: now reaches J7.2 (Pin_2)
- net AOUT7M: now also J17.2 (Pin_2)
- net AOUT6M: now reaches J7.3 (Pin_3)
- net AOUT6M: now also J16.2 (Pin_2)
- net AOUT5M: now reaches J7.4 (Pin_4)
- net AOUT5M: now also J15.2 (Pin_2)
- net AOUT4M: now reaches J7.5 (Pin_5)
- net AOUT4M: now also J14.2 (Pin_2)
- net AOUT3M: now reaches J7.6 (Pin_6)
- net AOUT3M: now also J13.2 (Pin_2)
- net AOUT2M: now reaches J7.7 (Pin_7)
- net AOUT2M: now also J12.2 (Pin_2)
- net AOUT1M: now reaches J7.8 (Pin_8)
- net AOUT1M: now also J11.2 (Pin_2)
- new net DOUT1M: J21.2 (Pin_2), J9.6 (Pin_6)
- new net DOUT2M: J22.2 (Pin_2), J9.8 (Pin_8)
- new net DOUT3M: J23.2 (Pin_2), J9.28 (Pin_28)
- no-connect marks 40 -> 29
Other:
- note added: "reserved for USB host shield"
- moved on the sheet: RN1, U7B, U7E
