File: PCB/motor-driver2022b/motor-driver2022b.kicad_pcb (KiCad board)
At the start: 2 copper layers, 142 x 134 mm, 114 parts, among them J1 Motor Power, J2 Logic Power, J3 Input Ch1, J4 Input Ch2, J5 Input Ch3, J6 Input Ch4, M1 Motor_DC, M2 Motor_DC, M3 Motor_DC, M4 Motor_DC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

Commit message: ガーバーデータを追加
git-svn-id: https://shiro-home.ddns.net/svn/project/motor-driver/trunk@45 73406841-da20-4056-b287-c5b29fcc9b8e
Other:
- rule pad_to_mask_clearance: 0.05 -> 0
