File: PCB/patch-board2022b/patch-board2022b.kicad_pcb (KiCad board)
At the start: 2 copper layers, 153 x 58 mm, 85 parts, among them J1 USB_B, J10 SERVO POWER SUPPLY, J11 AOUT1, J12 AOUT2, J13 AOUT3, J14 AOUT4, J15 AOUT5, J16 AOUT6, J17 AOUT7, J18 AOUT8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

Commit message: ガーバーデータを追加
git-svn-id: https://shiro-home.ddns.net/svn/project/motor-driver/trunk@48 73406841-da20-4056-b287-c5b29fcc9b8e
Other:
- rule pad_to_mask_clearance: 0.05 -> 0
