File: PCB/object-sensor2022a/object-sensor2022a-panelize4x1.kicad_pcb (KiCad board)
At the start: 2 copper layers, 50 x 78 mm, 40 parts, among them J1 Conn_01x03, U1 S6809

Commit message: ガーバーデータを追加
git-svn-id: https://shiro-home.ddns.net/svn/project/motor-driver/trunk@49 73406841-da20-4056-b287-c5b29fcc9b8e
Other:
- rule pad_to_mask_clearance: 0.05 -> 0
