File: trunk/PCB/object-sensor2022a/object-sensor2022a-panelize4x1.kicad_pcb (KiCad board)
At the start: 2 copper layers, 50 x 78 mm, 40 parts, among them J1 Conn_01x03, U1 S6809

Commit message: 面付けデータを修正
git-svn-id: https://shiro-home.ddns.net/svn/project/motor-driver@64 73406841-da20-4056-b287-c5b29fcc9b8e
Other:
- board size 50 x 78 mm -> 80 x 78 mm
